File: tia-rev1/tia-rev1.sch (EAGLE design)
At the start: 22 parts, among them IC1 TPS79850, IC2 OPA858, X2 SPAD, X3 SIGNAL_OUT, X4 VIN_PWR

Commit message: newest version
Connections:
- net N$2 renamed IN-
- net N$4 renamed TIA_FB
- net N$5 renamed V_OUT
- net N$7 renamed LDO_IN/EN
Changed lines of the file:
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@@
 </segment>
 </net>
-<net name="N$4" class="0">
+<net name="TIA_FB" class="0">
 <segment>
 <pinref part="IC2" gate="G$1" pin="FB"/>
@@
 </segment>
 </net>
-<net name="N$2" class="0">
+<net name="IN-" class="0">
 <segment>
 <pinref part="X2" gate="G1" pin="1"/>
@@
 </segment>
 </net>
-<net name="N$5" class="0">
+<net name="V_OUT" class="0">
 <segment>
 <pinref part="IC2" gate="G$1" pin="OUT"/>
@@
 </segment>
 </net>
-<net name="N$7" class="0">
+<net name="LDO_IN/EN" class="0">
 <segment>
 <pinref part="IC1" gate="G$1" pin="IN"/>
