File: tia-rev1/tia-rev1.brd (EAGLE design)
At the start: 38.1 x 25.4 mm, 22 parts, among them IC1 TPS79850, IC2 OPA858, X2 SPAD, X3 SIGNAL_OUT, X4 VIN_PWR

Commit message: newest version
Parts:
- moved C12 32.6 mm to (13.3, 17.9)
- moved X4 15.2 mm to (38.0, 20.2)
- moved X3 7.62 mm to (37.9, 5.08)
- moved R7 7.22 mm to (16.4, 15.2)
Connections:
- net N$2 renamed IN-
- net N$4 renamed TIA_FB
- net N$5 renamed V_OUT
- net N$7 renamed LDO_IN/EN
Routing:
- net IN-: track 0.00 -> 19.7 mm
- net LDO_IN/EN: track 2.03 -> 21.2 mm
- net V_OUT: track 1.05 -> 20.1 mm
- net TIA_FB: track 0.00 -> 5.66 mm
- net GND: track 9.52 -> 15.0 mm, vias 132 -> 108
- net VREF_2V5: track 20.9 -> 26.2 mm
- net PP_P5V0_ANALOG: track 50.1 -> 49.2 mm
- removed copper zone on layer 1, net NON_INV_OUT
Other:
- outline, holes or cut-outs redrawn

Commit message: newest version(again
Parts:
- moved C1 9.61 mm to (2.62, 22.4)
- moved C2 9.61 mm to (4.05, 22.4)
- moved C3 9.61 mm to (5.48, 22.4)
- moved IC1 9.61 mm to (8.97, 22.5)
- moved R1 9.61 mm to (6.91, 22.4)
- moved R3 9.61 mm to (6.27, 20.2)
- moved C4 9.61 mm to (15.8, 22.2)
- moved C8 9.61 mm to (15.8, 20.8)
- moved X4 8.34 mm to (29.7, 20.4)
- moved X3 8.34 mm to (29.5, 5.24)
- moved C12 2.76 mm to (13.8, 15.2), turned to 90 degrees
- turned R7 to 90 degrees
Routing:
- net PP_P5V0_ANALOG: track 49.2 -> 56.5 mm
- net V_OUT: track 20.1 -> 13.8 mm
- net GND: track 15.0 -> 21.1 mm, vias 108 -> 92
- net LDO_IN/EN: track 21.2 -> 25.7 mm
- net IN-: track 19.7 -> 15.3 mm
- net VREF_2V5: track 26.2 -> 27.3 mm
- net TIA_FB: track 5.66 -> 4.65 mm
- removed copper zone on layer 1, net INV_OUT
Other:
- board size 38.1 x 25.4 mm -> 29.8 x 25.6 mm
